File: esp8266bob.sch (KiCad schematic (older format))
At the start: 47 parts, among them P1 USB_OTG, P2 CONN_01X07, P3 CONN_01X07, P4 CONN_01X03, SW1 SW_PUSH, SW2 SW_PUSH, U1 TS 2940 CP33, U10 WS2812, U11 WS2812, U12 WS2812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

Commit message: gerber generated
Parts:
- added P5: CONN_01X03, Pin_Headers:Pin_Header_Straight_1x03, symbol CONN_01X03
Connections:
- wire segments 90 -> 91
- no-connect marks 8 -> 7
Changed lines of the file:
@@
 	1    0    0    -1
 $EndComp
-NoConn ~ 5200 6350
 Wire Wire Line
 	3100 1450 4200 1450
@@
 Wire Wire Line
 	5100 1350 5050 1350
+Wire Wire Line
+	5200 6350 5350 6350
+$Comp
+L CONN_01X03 P5
+U 1 1 56F1F05C
+P 5550 6350
+F 0 "P5" H 5550 6550 50  0000 C CNN
+F 1 "CONN_01X03" V 5650 6350 50  0000 C CNN
+F 2 "Pin_Headers:Pin_Header_Straight_1x03" H 5550 6350 50  0001 C CNN
+F 3 "" H 5550 6350 50  0000 C CNN
+	1    5550 6350
+	1    0    0    -1
+$EndComp
+$Comp
+L +5V #PWR049
+U 1 1 56F1F0EB
+P 5350 6250
+F 0 "#PWR049" H 5350 6100 50  0001 C CNN
+F 1 "+5V" H 5350 6390 50  0000 C CNN
+F 2 "" H 5350 6250 50  0000 C CNN
+F 3 "" H 5350 6250 50  0000 C CNN
+	1    5350 6250
+	1    0    0    -1
+$EndComp
+$Comp
+L GND #PWR050
+U 1 1 56F1F3D4
+P 5350 6450
+F 0 "#PWR050" H 5350 6200 50  0001 C CNN
+F 1 "GND" H 5350 6300 50  0000 C CNN
+F 2 "" H 5350 6450 50  0000 C CNN
+F 3 "" H 5350 6450 50  0000 C CNN
+	1    5350 6450
+	1    0    0    -1
+$EndComp
 $EndSCHEMATC

Commit message: bugs fixed in the schematic
Parts:
- added R? (x2): 10k, symbol R
Connections:
- net labels added: GPIO2
- net labels removed: Prog_pin
- wire segments 91 -> 94
Changed lines of the file:
@@
 $EndComp
 Text Label 8500 4200 0    60   ~ 0
-Prog_pin
+GPIO2
 $Comp
 L GND #PWR06
@@
 $EndComp
 Text Label 4650 1750 0    60   ~ 0
+CH340_RX
+Text Label 4650 1550 0    60   ~ 0
 CH340_TX
-Text Label 4650 1550 0    60   ~ 0
-CH340_RX
 $Comp
 L JUMPER JP1
@@
 RESET
 Text Label 9900 4300 0    60   ~ 0
-Prog_pin
+GPIO0
 $Comp
 L GND #PWR041
@@
 GPIO0
 Text Label 8100 2350 0    60   ~ 0
-Prog_pin
+GPIO2
 Text Label 8100 2450 0    60   ~ 0
 GPIO15
@@
 	8750 4100 8500 4100
 Wire Wire Line
-	8750 4200 8500 4200
+	8500 4200 8950 4200
 Wire Wire Line
 	8750 4300 8500 4300
@@
 	1450 2350 1450 2550
 Connection ~ 1450 2550
-Connection ~ 10400 5550
 $Comp
 L CONN_01X07 P3
@@
 	1    0    0    -1
 $EndComp
+$Comp
+L R R?
+U 1 1 570591ED
+P 10200 4150
+F 0 "R?" V 10280 4150 50  0000 C CNN
+F 1 "10k" V 10200 4150 50  0000 C CNN
+F 2 "" V 10130 4150 50  0000 C CNN
+F 3 "" H 10200 4150 50  0000 C CNN
+	1    10200 4150
+	1    0    0    -1
+$EndComp
+Connection ~ 10200 4300
+$Comp
+L +3V3 #PWR?
+U 1 1 57059540
+P 10200 3950
+F 0 "#PWR?" H 10200 3800 50  0001 C CNN
+F 1 "+3V3" H 10200 4090 50  0000 C CNN
+F 2 "" H 10200 3950 50  0000 C CNN
+F 3 "" H 10200 3950 50  0000 C CNN
+	1    10200 3950
+	0    1    1    0
+$EndComp
+Wire Wire Line
+	10200 3950 10200 4000
+Wire Wire Line
+	8950 4200 8950 4350
+$Comp
+L R R?
+U 1 1 57059B68
+P 8950 4500
+F 0 "R?" V 9030 4500 50  0000 C CNN
+F 1 "10k" V 8950 4500 50  0000 C CNN
+F 2 "" V 8880 4500 50  0000 C CNN
+F 3 "" H 8950 4500 50  0000 C CNN
+	1    8950 4500
+	1    0    0    -1
+$EndComp
+$Comp
+L +3V3 #PWR?
+U 1 1 57059C43
+P 8950 4700
+F 0 "#PWR?" H 8950 4550 50  0001 C CNN
+F 1 "+3V3" H 8950 4840 50  0000 C CNN
+F 2 "" H 8950 4700 50  0000 C CNN
+F 3 "" H 8950 4700 50  0000 C CNN
+	1    8950 4700
+	-1   0    0    1
+$EndComp
+Wire Wire Line
+	8950 4650 8950 4700
 $EndSCHEMATC

Commit message: bugfixes, auto programming pins connected
Parts:
- removed R?: 10k, symbol R
- added JP3, JP4: JUMPER, open-project:S_JUMPER_2, symbol JUMPER
- added R5: 10k, Resistors_SMD:R_0603_HandSoldering, symbol R
- R6: renamed from R?; footprint (none) -> Resistors_SMD:R_0603_HandSoldering
Connections:
- net labels added: DTR, RTS, reset
- wire segments 94 -> 99
- no-connect marks 7 -> 5
Other:
- moved on the sheet: P2, P3
